Commit message: feat: implement aggressive driver model with lidar-based avoidance and auto-reset supervisor

File: src/adas_project/urdf/vehicle.xacro (robot description, xacro)
@@ -81,5 +81,5 @@
         <origin xyz="${x} ${y} ${z}"/>
         <axis xyz="0 1 0"/>
-        <limit effort="500.0" velocity="20.0"/>
+        <limit effort="500.0" velocity="150.0"/>
       </joint>
     </xacro:unless>
@@ -99,5 +99,5 @@
     <parent link="chassis"/>
     <child link="lidar_link"/>
-    <origin xyz="0.4 0 0.15" rpy="0 0 0"/>
+    <origin xyz="0.4 0 0.5" rpy="0 0 0"/>
   </joint>
   <!-- Camera -->
@@ -137,4 +137,8 @@
       <rear_left_joint>rear_left_wheel_joint</rear_left_joint>
       <rear_right_joint>rear_right_wheel_joint</rear_right_joint>
+      <!-- Kinematics -->
+      <wheel_separation>0.6</wheel_separation>
+      <wheel_base>0.8</wheel_base>
+      <wheel_diameter>0.3</wheel_diameter>
       <!-- Geometry -->
       <max_steer>0.6</max_steer>
@@ -182,6 +186,6 @@
         </scan>
         <range>
-          <min>0.15</min>
-          <max>50.0</max>
+          <min>0.8</min>
+          <max>100.0</max>
         </range>
       </ray>
